File: hardware/electronics/EagleFiles/placa.brd (EAGLE design)
At the start: 160 x 100 mm, 26 parts, among them IC1 1182-A4988, IC2 1182-A4988, IC3 1182-A4988, IC4 1182-A4988, IC5 1182-A4988, IC6 1182-A4988

Commit message: eagle files
Parts:
- moved C3 181.5 mm to (100.3, 87.6), turned to 270 degrees
- moved SV13 167.9 mm to (102.9, 53.3)
- moved SV12 158.0 mm to (99.1, 26.7), turned to 270 degrees
- moved IC3 154.8 mm to (87.6, 74.9)
- moved C2 144.6 mm to (71.1, 87.6), turned to 270 degrees
- moved C7 141.0 mm to (100.3, 39.4), turned to 270 degrees
- moved SV5 140.0 mm to (77.5, 80.0), turned to 90 degrees
- moved IC6 126.5 mm to (87.6, 26.7)
- moved SV11 123.3 mm to (77.5, 31.8), turned to 90 degrees
- moved SV9 119.6 mm to (48.3, 31.8), turned to 90 degrees
- moved SV6 119.4 mm to (99.1, 74.9), turned to 270 degrees
- moved SV4 118.2 mm to (69.8, 74.9), turned to 270 degrees
- moved IC2 114.2 mm to (58.4, 74.9)
- moved C1 109.3 mm to (41.9, 87.6), turned to 270 degrees
- moved SV10 106.8 mm to (69.8, 26.7), turned to 270 degrees
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Connections:
- net 0 renamed GND
- net MOTOR1DIR: now also JP1.2; no longer JP1.1
- net MOTOR1STEP: now also JP1.1; no longer JP1.2
- net MOTOR2DIR: now also JP1.4; no longer JP1.3
- net MOTOR2STEP: now also JP1.3; no longer JP1.4
- net MOTOR3DIR: now also JP1.6; no longer JP1.5
- net MOTOR3STEP: now also JP1.5; no longer JP1.6
- net MOTOR4DIR: now also JP1.8; no longer JP1.7
- net MOTOR4STEP: now also JP1.7; no longer JP1.8
- net MOTOR5DIR: now also JP1.10; no longer JP1.9
- net MOTOR5STEP: now also JP1.9; no longer JP1.10
- net MOTOR6DIR: now also JP1.12; no longer JP1.11
- net MOTOR6STEP: now also JP1.11; no longer JP1.12
Routing:
- net LOGICVIN: track 0.00 -> 364.3 mm
- net MOTORVIN: track 0.00 -> 237.3 mm
- net MOTOR4DIR: track 0.00 -> 66.7 mm
- net MOTOR4STEP: track 0.00 -> 62.3 mm
- net MOTOR6DIR: track 0.00 -> 45.9 mm
- net MOTOR5DIR: track 0.00 -> 41.0 mm
- net MOTOR6STEP: track 0.00 -> 39.3 mm
- net MOTOR3STEP: track 0.00 -> 37.5 mm
- net MOTOR5STEP: track 0.00 -> 37.4 mm
- net MOTOR3DIR: track 0.00 -> 33.9 mm
- net MOTOR1STEP: track 0.00 -> 32.1 mm
- net MOTOR1DIR: track 0.00 -> 29.3 mm
- net MOTOR2STEP: track 0.00 -> 17.9 mm
- net MOTOR2DIR: track 0.00 -> 14.3 mm
- net N$9: track 0.00 -> 5.08 mm
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- added copper zone on layer 1, net GND
Other:
- board size 160 x 100 mm -> 99 x 82.2 mm
