File: hardware/electronics/EagleFiles/placa.sch (EAGLE design)
At the start: 26 parts, among them IC1 1182-A4988, IC2 1182-A4988, IC3 1182-A4988, IC4 1182-A4988, IC5 1182-A4988, IC6 1182-A4988

Commit message: eagle files
Connections:
- net 0 renamed GND
- net MOTOR1DIR: now also JP1.2; no longer JP1.1
- net MOTOR1STEP: now also JP1.1; no longer JP1.2
- net MOTOR2DIR: now also JP1.4; no longer JP1.3
- net MOTOR2STEP: now also JP1.3; no longer JP1.4
- net MOTOR3DIR: now also JP1.6; no longer JP1.5
- net MOTOR3STEP: now also JP1.5; no longer JP1.6
- net MOTOR4DIR: now also JP1.8; no longer JP1.7
- net MOTOR4STEP: now also JP1.7; no longer JP1.8
- net MOTOR5DIR: now also JP1.10; no longer JP1.9
- net MOTOR5STEP: now also JP1.9; no longer JP1.10
- net MOTOR6DIR: now also JP1.12; no longer JP1.11
- net MOTOR6STEP: now also JP1.11; no longer JP1.12
